Commit message: New package name

File: urdf/ackermann.xacro (robot description, xacro)
@@ -1,5 +1,5 @@
 <?xml version="1.0" ?>
 <robot name="robot" xmlns:xacro="http://ros.org/wiki/xacro">
-  <xacro:property name="package_name" value="ackermann_slam_sim"/>
+  <xacro:property name="package_name" value="slam_sim"/>
   <xacro:property name="PI" value="3.14159265"/>
   <xacro:property name="L_x" value="0.4"/> <!-- Robot X axis (front-back) -->

File: urdf/sensors_diffbot.xacro (robot description, xacro)
@@ -1,5 +1,5 @@
 <?xml version="1.0"?>
 <robot name="robot" xmlns:xacro="http://ros.org/wiki/xacro">
-  <xacro:property name="package_name" value="ackermann_slam_sim"/>
+  <xacro:property name="package_name" value="slam_sim"/>
   <xacro:property name="PI" value="3.14159265"/>
   <xacro:property name="wheelSeparation" value="0.13"/>

Commit message: Extrinsect Warning update

File: urdf/ackermann.xacro (robot description, xacro)
@@ -21,4 +21,5 @@
   <xacro:arg name="max_distance"    default="100.0"/>
   <xacro:arg name="resolution"    default="0.017453"/>
+  <xacro:arg name="lidar_origin_joint"    default="-0.04 0 0.07"/>
   <xacro:arg name="imu_frequency"    default="50"/>
   <!-- Custom color (for Ign and RViz) -->
@@ -168,5 +169,5 @@
     <parent link="base_link"/>
     <child link="lidar_link"/>
-    <origin xyz="-0.04 0 0.07" rpy="0 0 0"/>
+    <origin xyz=$(arg lidar_origin_joint) rpy="0 0 0"/>
   </joint>
   <link name="lidar_link">

File: urdf/sensors_diffbot.xacro (robot description, xacro)
@@ -20,4 +20,5 @@
   <xacro:arg name="max_distance"    default="100.0"/>
   <xacro:arg name="resolution"    default="0.017453"/>
+  <xacro:arg name="lidar_origin_joint"    default="-0.04 0 0.07"/>
   <xacro:arg name="imu_frequency"    default="50"/>
   <!-- Custom color (for Ign and RViz) -->
@@ -250,5 +251,5 @@
     <parent link="base_link"/>
     <child link="lidar_link"/>
-    <origin xyz="-0.04 0 0.07" rpy="0 0 0"/>
+    <origin xyz=$(arg lidar_origin_joint) rpy="0 0 0"/>
   </joint>
   <link name="lidar_link">

Commit message: Bug fixed

File: urdf/ackermann.xacro (robot description, xacro)
@@ -21,5 +21,4 @@
   <xacro:arg name="max_distance"    default="100.0"/>
   <xacro:arg name="resolution"    default="0.017453"/>
-  <xacro:arg name="lidar_origin_joint"    default="-0.04 0 0.07"/>
   <xacro:arg name="imu_frequency"    default="50"/>
   <!-- Custom color (for Ign and RViz) -->
@@ -169,5 +168,5 @@
     <parent link="base_link"/>
     <child link="lidar_link"/>
-    <origin xyz=$(arg lidar_origin_joint) rpy="0 0 0"/>
+    <origin xyz="-0.04 0 0.07" rpy="0 0 0"/>
   </joint>
   <link name="lidar_link">

File: urdf/sensors_diffbot.xacro (robot description, xacro)
@@ -20,5 +20,4 @@
   <xacro:arg name="max_distance"    default="100.0"/>
   <xacro:arg name="resolution"    default="0.017453"/>
-  <xacro:arg name="lidar_origin_joint"    default="-0.04 0 0.07"/>
   <xacro:arg name="imu_frequency"    default="50"/>
   <!-- Custom color (for Ign and RViz) -->
@@ -251,5 +250,5 @@
     <parent link="base_link"/>
     <child link="lidar_link"/>
-    <origin xyz=$(arg lidar_origin_joint) rpy="0 0 0"/>
+    <origin xyz="-0.04 0 0.07" rpy="0 0 0"/>
   </joint>
   <link name="lidar_link">
